File: quantar_breakout_v0.0.1.kicad_sch (KiCad schematic)
At the start: 5 parts, among them J1 DE9_Pins, J2 AudioPlug2, J3 AudioPlug2, J4 Conn_02x20_Odd_Even, U1 FXMA108

Commit message: Remove old stuff
Parts:
- removed J1: DE9_Pins, symbol Connector:DE9_Pins
- removed J2, J3: AudioPlug2, symbol Connector_Audio:AudioPlug2
- removed J4: Conn_02x20_Odd_Even, symbol Connector_Generic:Conn_02x20_Odd_Even
- removed U1: FXMA108, Package_DFN_QFN:WQFN-20-1EP_2.5x4.5mm_P0.5mm_EP1x2.9mm, symbol Logic_LevelTranslator:FXMA108
